File: iPod nano 6 LCD.sch (KiCad schematic (older format))
At the start: 5 parts, among them U1 AP5724

Commit message: Add schematic symbol for the Molex connector for the display
Parts:
- added J?: Molex_503548-1220, symbol iPod~nano~6~LCD:Molex_503548-1220
Connections:
- net labels added: CLKN, CLKP, DN, DP, RESET, SYNC, VDD, VEE
- wire segments 26 -> 30
Other:
- note added: "Display connector"
Changed lines of the file:
@@
 Text GLabel 1850 1150 2    50   Input ~ 0
 LEDPWM
-Text Notes 600  2350 0    50   ~ 0
+Text Notes 600  2400 0    50   ~ 0
 Power generation for backlight.\nSchematic kindly provided by Mike "Electric Stuff" Harrison\nelectricstuff.co.uk\n
 Wire Notes Line
-	550  2450 3250 2450
+	3250 2450 3250 550
+$Comp
+L iPod~nano~6~LCD:Molex_503548-1220 J?
+U 1 1 5FD66C40
+P 4000 1100
+F 0 "J?" H 4000 1450 50  0000 L CNN
+F 1 "Molex_503548-1220" H 3900 150 50  0000 L CNN
+F 2 "" H 4000 1100 50  0001 C CNN
+F 3 "" H 4000 1100 50  0001 C CNN
+	1    4000 1100
+	1    0    0    -1
+$EndComp
+Text GLabel 3900 850  0    50   Input ~ 0
+CLKP
+Text GLabel 3900 950  0    50   Input ~ 0
+VDD
+Text GLabel 3900 1050 0    50   Input ~ 0
+CLKN
+Text GLabel 3900 1150 0    50   Input ~ 0
+VEE
+Text GLabel 3900 1350 0    50   Input ~ 0
+SYNC
+Text GLabel 3900 1450 0    50   Input ~ 0
+DP
+Text GLabel 3900 1550 0    50   Input ~ 0
+RESET
+Text GLabel 3900 1650 0    50   Input ~ 0
+DN
+Text GLabel 3900 1750 0    50   Input ~ 0
+LED+
+Text GLabel 3900 1950 0    50   Input ~ 0
+LED-
+Wire Wire Line
+	3900 1250 3550 1250
+Wire Wire Line
+	3550 1250 3550 1300
+Wire Wire Line
+	3900 1850 3550 1850
+Wire Wire Line
+	3550 1850 3550 1900
+$Comp
+L power:GND #PWR?
+U 1 1 5FD68A93
+P 3550 1900
+F 0 "#PWR?" H 3550 1650 50  0001 C CNN
+F 1 "GND" H 3555 1727 50  0000 C CNN
+F 2 "" H 3550 1900 50  0001 C CNN
+F 3 "" H 3550 1900 50  0001 C CNN
+	1    3550 1900
+	1    0    0    -1
+$EndComp
+$Comp
+L power:GND #PWR?
+U 1 1 5FD68B8D
+P 3550 1300
+F 0 "#PWR?" H 3550 1050 50  0001 C CNN
+F 1 "GND" H 3555 1127 50  0000 C CNN
+F 2 "" H 3550 1300 50  0001 C CNN
+F 3 "" H 3550 1300 50  0001 C CNN
+	1    3550 1300
+	1    0    0    -1
+$EndComp
 Wire Notes Line
-	3250 2450 3250 550
+	4800 2450 4800 550
+Wire Notes Line
+	550  2450 4800 2450
+Text Notes 3300 2400 0    50   ~ 0
+Display connector
 $EndSCHEMATC

Commit message: Add USB and ATSAMD processor
Parts:
- added C1, C10, C11, C12, C14, C2, C3, C4, C5, C6, C7, C8, C9: 1u, Capacitor_SMD:C_0603_1608Metric, symbol Device:C_Small
- added C15: .1u, Capacitor_SMD:C_0603_1608Metric, symbol Device:C_Small
- added C16, C17: 10u, Capacitor_SMD:C_0603_1608Metric, symbol Device:C_Small
- added D2: +5V, LED_SMD:LED_0603_1608Metric, symbol Device:LED_Small
- added D3: +1.8V, LED_SMD:LED_0603_1608Metric, symbol Device:LED_Small
- added D4: +3.3v, LED_SMD:LED_0603_1608Metric, symbol Device:LED_Small
- added J2: USB_C_Receptacle_USB2.0, iPod nano 6 LCD:USB_C_Receptacle_GT-USB-7010, symbol Connector:USB_C_Receptacle_USB2.0
- added L3: 2.2uH, Inductor_SMD:L_0603_1608Metric, symbol Device:L
- added R3: 100, Resistor_SMD:R_0603_1608Metric, symbol Device:R_Small
- added R4: 16, Resistor_SMD:R_0603_1608Metric, symbol Device:R_Small
- added R5: 8, Resistor_SMD:R_0603_1608Metric, symbol Device:R_Small
- added U2: ATSAM3SD8BA-AU, iPod nano 6 LCD:QFP-64_12x12_Pitch0.5mm, symbol iPod~nano~6~LCD:ATSAM3SD8BA-AU
- added U3: AZ1117-1.8, Package_TO_SOT_SMD:SOT-223-3_TabPin2, symbol Regulator_Linear:AZ1117-1.8
- added U4: TPS63001, Package_SON:Texas_DRC0010J_ThermalVias, symbol Regulator_Switching:TPS63002
- gave numbers to parts that had none: 1
Connections:
- net labels added: +1V8, +3.3V, +5V, VDDIN, VDDOUT, VDDPLL
- net labels removed: +3V0
- wire segments 30 -> 120
Other:
- note added: "BL Generator supply voltage"
- note added: "Main CPU power reg"
- note added: "Some of the CPU decoupling\n"

Commit message: Add JTAG and LCD connector and bias resistors
Parts:
- added J3: Conn_01x06_Male, Connector_JST:JST_GH_BM06B-GHS-TBT_1x06-1MP_P1.25mm_Vertical, symbol Connector_Generic_MountingPin:Conn_01x06_MountingPin
- added R10, R12, R14, R9: 47, Resistor_SMD:R_0603_1608Metric, symbol Device:R_Small
- added R11, R13, R7, R8: 220, Resistor_SMD:R_0603_1608Metric, symbol Device:R_Small
- added R6: 10k, Resistor_SMD:R_0603_1608Metric, symbol Device:R_Small
- J1: footprint (none) -> iPod nano 6 LCD:Molex 503548-1220
Connections:
- net labels added: IC_CLKN, IC_CLKP, TCK, TDI, TDO, TMS
- net labels removed: RESET, VDD, VEE
- wire segments 120 -> 146

Commit message: Add the 2 crystals on board
Parts:
- added C13, C18: 12.5p, Capacitor_SMD:C_0603_1608Metric, symbol Device:C_Small
- added C? (x2): 10p, Capacitor_SMD:C_0603_1608Metric, symbol Device:C_Small
- added Y1: 32.768k, Crystal:Crystal_SMD_Abracon_ABS25-4Pin_8.0x3.8mm, symbol Device:Crystal_Small
- added Y?: 20MHz, Crystal:Crystal_SMD_Abracon_ABM8G-4Pin_3.2x2.5mm, symbol Device:Crystal_Small
Connections:
- wire segments 146 -> 168
Changed lines of the file:
@@
 P 950 9650
 AR Path="/5FEB2752/5FEFBAAD" Ref="#PWR?"  Part="1"
-AR Path="/5FEFBAAD" Ref="#PWR?"  Part="1"
-F 0 "#PWR?" H 950 9400 50  0001 C CNN
+AR Path="/5FEFBAAD" Ref="#PWR0115"  Part="1"
+F 0 "#PWR0115" H 950 9400 50  0001 C CNN
 F 1 "GND" H 955 9477 50  0000 C CNN
 F 2 "" H 950 9650 50  0001 C CNN
@@
 	1    0    0    -1
 $EndComp
+$Comp
+L Device:Crystal_Small Y1
+U 1 1 5FF05C66
+P 8750 2450
+F 0 "Y1" V 8704 2538 50  0000 L CNN
+F 1 "32.768k" V 8900 2300 50  0000 L CNN
+F 2 "Crystal:Crystal_SMD_Abracon_ABS25-4Pin_8.0x3.8mm" H 8750 2450 50  0001 C CNN
+F 3 "~" H 8750 2450 50  0001 C CNN
+	1    8750 2450
+	0    1    1    0
+$EndComp
+Wire Wire Line
+	8500 2400 8500 2350
+Wire Wire Line
+	8500 2350 8750 2350
+Wire Wire Line
+	8400 2400 8500 2400
+Wire Wire Line
+	8400 2500 8500 2500
+Wire Wire Line
+	8500 2500 8500 2550
+Wire Wire Line
+	8500 2550 8750 2550
+Connection ~ 8750 2350
+Connection ~ 8750 2550
+$Comp
+L Device:C_Small C13
+U 1 1 5FF208F8
+P 9050 2350
+F 0 "C13" H 8959 2304 50  0000 R CNN
+F 1 "12.5p" H 8959 2395 50  0000 R CNN
+F 2 "Capacitor_SMD:C_0603_1608Metric" H 9050 2350 50  0001 C CNN
+F 3 "~" H 9050 2350 50  0001 C CNN
+	1    9050 2350
+	0    -1   1    0
+$EndComp
+$Comp
+L Device:C_Small C18
+U 1 1 5FF20D1C
+P 9050 2550
+F 0 "C18" H 8959 2504 50  0000 R CNN
+F 1 "12.5p" H 8959 2595 50  0000 R CNN
+F 2 "Capacitor_SMD:C_0603_1608Metric" H 9050 2550 50  0001 C CNN
+F 3 "~" H 9050 2550 50  0001 C CNN
+	1    9050 2550
+	0    -1   -1   0
+$EndComp
+Wire Wire Line
+	8750 2350 8950 2350
+Wire Wire Line
+	8950 2550 8750 2550
+Wire Wire Line
+	9150 2550 9200 2550
+Wire Wire Line
+	9200 2550 9200 2350
+Wire Wire Line
+	9200 2350 9150 2350
+$Comp
+L power:GND #PWR0116
+U 1 1 5FF353AF
+P 9200 2550
+F 0 "#PWR0116" H 9200 2300 50  0001 C CNN
+F 1 "GND" H 9300 2450 50  0000 C CNN
+F 2 "" H 9200 2550 50  0001 C CNN
+F 3 "" H 9200 2550 50  0001 C CNN
+	1    9200 2550
+	1    0    0    -1
+$EndComp
+Connection ~ 9200 2550
+$Comp
+L Device:Crystal_Small Y?
+U 1 1 5FF4687B
+P 8750 5950
+F 0 "Y?" V 8704 6038 50  0000 L CNN
+F 1 "20MHz" V 8900 5800 50  0000 L CNN
+F 2 "Crystal:Crystal_SMD_Abracon_ABM8G-4Pin_3.2x2.5mm" H 8750 5950 50  0001 C CNN
+F 3 "~" H 8750 5950 50  0001 C CNN
+	1    8750 5950
+	0    1    1    0
+$EndComp
+Wire Wire Line
+	8500 5900 8500 5850
+Wire Wire Line
+	8500 5850 8750 5850
+Wire Wire Line
+	8400 5900 8500 5900
+Wire Wire Line
+	8400 6000 8500 6000
+Wire Wire Line
+	8500 6000 8500 6050
+Wire Wire Line
+	8500 6050 8750 6050
+Connection ~ 8750 5850
+Connection ~ 8750 6050
+$Comp
+L Device:C_Small C?
+U 1 1 5FF46889
+P 9050 5850
+F 0 "C?" H 8959 5804 50  0000 R CNN
+F 1 "10p" H 8959 5895 50  0000 R CNN
+F 2 "Capacitor_SMD:C_0603_1608Metric" H 9050 5850 50  0001 C CNN
+F 3 "~" H 9050 5850 50  0001 C CNN
+	1    9050 5850
+	0    -1   1    0
+$EndComp
+$Comp
+L Device:C_Small C?
+U 1 1 5FF4688F
+P 9050 6050
+F 0 "C?" H 8959 6004 50  0000 R CNN
+F 1 "10p" H 8959 6095 50  0000 R CNN
+F 2 "Capacitor_SMD:C_0603_1608Metric" H 9050 6050 50  0001 C CNN
+F 3 "~" H 9050 6050 50  0001 C CNN
+	1    9050 6050
+	0    -1   -1   0
+$EndComp
+Wire Wire Line
+	8750 5850 8950 5850
+Wire Wire Line
+	8950 6050 8750 6050
+Wire Wire Line
+	9150 6050 9200 6050
+Wire Wire Line
+	9200 6050 9200 5850
+Wire Wire Line
+	9200 5850 9150 5850
+$Comp
+L power:GND #PWR?
+U 1 1 5FF4689A
+P 9200 6050
+F 0 "#PWR?" H 9200 5800 50  0001 C CNN
+F 1 "GND" H 9300 5950 50  0000 C CNN
+F 2 "" H 9200 6050 50  0001 C CNN
+F 3 "" H 9200 6050 50  0001 C CNN
+	1    9200 6050
+	1    0    0    -1
+$EndComp
+Connection ~ 9200 6050
 $EndSCHEMATC

Commit message: Save anotated crystal schematic
Parts:
- gave numbers to parts that had none: 3
Changed lines of the file:
@@
 Connection ~ 9200 2550
 $Comp
-L Device:Crystal_Small Y?
+L Device:Crystal_Small Y2
 U 1 1 5FF4687B
 P 8750 5950
-F 0 "Y?" V 8704 6038 50  0000 L CNN
+F 0 "Y2" V 8704 6038 50  0000 L CNN
 F 1 "20MHz" V 8900 5800 50  0000 L CNN
 F 2 "Crystal:Crystal_SMD_Abracon_ABM8G-4Pin_3.2x2.5mm" H 8750 5950 50  0001 C CNN
@@
 Connection ~ 8750 6050
 $Comp
-L Device:C_Small C?
+L Device:C_Small C19
 U 1 1 5FF46889
 P 9050 5850
-F 0 "C?" H 8959 5804 50  0000 R CNN
+F 0 "C19" H 8959 5804 50  0000 R CNN
 F 1 "10p" H 8959 5895 50  0000 R CNN
 F 2 "Capacitor_SMD:C_0603_1608Metric" H 9050 5850 50  0001 C CNN
@@
 $EndComp
 $Comp
-L Device:C_Small C?
+L Device:C_Small C20
 U 1 1 5FF4688F
 P 9050 6050
-F 0 "C?" H 8959 6004 50  0000 R CNN
+F 0 "C20" H 8959 6004 50  0000 R CNN
 F 1 "10p" H 8959 6095 50  0000 R CNN
 F 2 "Capacitor_SMD:C_0603_1608Metric" H 9050 6050 50  0001 C CNN
@@
 	9200 5850 9150 5850
 $Comp
-L power:GND #PWR?
+L power:GND #PWR020
 U 1 1 5FF4689A
 P 9200 6050
-F 0 "#PWR?" H 9200 5800 50  0001 C CNN
+F 0 "#PWR020" H 9200 5800 50  0001 C CNN
 F 1 "GND" H 9300 5950 50  0000 C CNN
 F 2 "" H 9200 6050 50  0001 C CNN

Commit message: Add Symbol for XTSD04GLGEAG
Parts:
- added C21: 1u, Capacitor_SMD:C_0603_1608Metric, symbol Device:C_Small
- added U5: XTSD04GLGEAG, symbol iPod~nano~6~LCD:XTSD04GLGEAG
Connections:
- net labels added: MISO, MOSI, SCLK, SD_CS
- wire segments 168 -> 172
Other:
- note added: "4GB Flash module using SPI & SD Card protocol"
- note added: "BL Generator & SPI FLASH supply voltage"
- note removed: "BL Generator supply voltage"
Changed lines of the file:
@@
 	3250 550  3250 6200
 Text Notes 550  6150 0    50   ~ 0
-BL Generator supply voltage
+BL Generator & SPI FLASH supply voltage
 $Comp
 L Regulator_Linear:AZ1117-1.8 U3
@@
 $EndComp
 Connection ~ 9200 6050
+$Comp
+L iPod~nano~6~LCD:XTSD04GLGEAG U5
+U 1 1 5FE33365
+P 14900 1300
+F 0 "U5" H 15100 750 50  0000 L CNN
+F 1 "XTSD04GLGEAG" H 14650 650 50  0000 L CNN
+F 2 "" H 14900 1300 50  0001 C CNN
+F 3 "" H 14900 1300 50  0001 C CNN
+	1    14900 1300
+	1    0    0    -1
+$EndComp
+$Comp
+L Device:C_Small C21
+U 1 1 5FE33CAA
+P 14150 950
+F 0 "C21" H 14059 904 50  0000 R CNN
+F 1 "1u" H 14059 995 50  0000 R CNN
+F 2 "Capacitor_SMD:C_0603_1608Metric" H 14150 950 50  0001 C CNN
+F 3 "~" H 14150 950 50  0001 C CNN
+	1    14150 950
+	1    0    0    1
+$EndComp
+Wire Wire Line
+	14150 850  14150 800
+Connection ~ 14150 850
+Wire Wire Line
+	14150 1050 14150 1100
+Connection ~ 14150 1050
+$Comp
+L power:GND #PWR022
+U 1 1 5FE5BCCD
+P 14150 1100
+F 0 "#PWR022" H 14150 850 50  0001 C CNN
+F 1 "GND" H 14155 927 50  0000 C CNN
+F 2 "" H 14150 1100 50  0001 C CNN
+F 3 "" H 14150 1100 50  0001 C CNN
+	1    14150 1100
+	1    0    0    -1
+$EndComp
+$Comp
+L power:+3.3V #PWR021
+U 1 1 5FE73C49
+P 14150 800
+F 0 "#PWR021" H 14150 650 50  0001 C CNN
+F 1 "+3.3V" H 14165 973 50  0000 C CNN
+F 2 "" H 14150 800 50  0001 C CNN
+F 3 "" H 14150 800 50  0001 C CNN
+	1    14150 800
+	1    0    0    -1
+$EndComp
+Text GLabel 14550 1300 0    50   Input ~ 0
+SD_CS
+Wire Wire Line
+	14150 1050 14550 1050
+Wire Wire Line
+	14150 850  14550 850
+Text GLabel 14550 1400 0    50   Input ~ 0
+SCLK
+Text GLabel 14550 1500 0    50   Input ~ 0
+MOSI
+Text GLabel 14550 1600 0    50   Input ~ 0
+MISO
+Wire Notes Line
+	13500 500  13500 2150
+Wire Notes Line
+	13500 2150 16000 2150
+Text Notes 13550 2100 0    50   ~ 0
+4GB Flash module using SPI & SD Card protocol
 $EndSCHEMATC

Commit message: Add Footprint for the flash
Parts:
- U5: footprint (none) -> iPod nano 6 LCD:XTSD04GLGEAG
Changed lines of the file:
@@
 F 0 "U5" H 15100 750 50  0000 L CNN
 F 1 "XTSD04GLGEAG" H 14650 650 50  0000 L CNN
-F 2 "" H 14900 1300 50  0001 C CNN
+F 2 "iPod nano 6 LCD:XTSD04GLGEAG" H 14900 1300 50  0001 C CNN
 F 3 "" H 14900 1300 50  0001 C CNN
 	1    14900 1300

Commit message: Lets do some routing changes: Unroute all!
Parts:
- added D?: +3.3v, LED_SMD:LED_0603_1608Metric, symbol Device:LED_Small
- added R?: 8, Resistor_SMD:R_0603_1608Metric, symbol Device:R_Small
Connections:
- wire segments 172 -> 175
Other:
- note added: "Create 1.8V for the lcd"
- note added: "Main power"
- note removed: "BL Generator & SPI FLASH supply voltage"
- note removed: "Main CPU power reg"
Changed lines of the file:
@@
 Wire Wire Line
 	6750 3950 6600 3950
-$Comp
-L power:+1V8 #PWR011
-U 1 1 5FE001DC
-P 6500 2550
-F 0 "#PWR011" H 6500 2400 50  0001 C CNN
-F 1 "+1V8" H 6350 2600 50  0000 C CNN
-F 2 "" H 6500 2550 50  0001 C CNN
-F 3 "" H 6500 2550 50  0001 C CNN
-	1    6500 2550
-	1    0    0    -1
-$EndComp
-$Comp
-L power:+1V8 #PWR012
-U 1 1 5FE0092F
-P 6500 2900
-F 0 "#PWR012" H 6500 2750 50  0001 C CNN
-F 1 "+1V8" H 6350 2950 50  0000 C CNN
-F 2 "" H 6500 2900 50  0001 C CNN
-F 3 "" H 6500 2900 50  0001 C CNN
-	1    6500 2900
-	1    0    0    -1
-$EndComp
 Wire Wire Line
 	6500 2950 6500 2900
 Connection ~ 6500 2950
-$Comp
-L power:+1V8 #PWR013
-U 1 1 5FE01697
-P 6500 3300
-F 0 "#PWR013" H 6500 3150 50  0001 C CNN
-F 1 "+1V8" H 6350 3350 50  0000 C CNN
-F 2 "" H 6500 3300 50  0001 C CNN
-F 3 "" H 6500 3300 50  0001 C CNN
-	1    6500 3300
-	1    0    0    -1
-$EndComp
-$Comp
-L power:+1V8 #PWR014
-U 1 1 5FE01A30
-P 6500 3700
-F 0 "#PWR014" H 6500 3550 50  0001 C CNN
-F 1 "+1V8" H 6350 3750 50  0000 C CNN
-F 2 "" H 6500 3700 50  0001 C CNN
-F 3 "" H 6500 3700 50  0001 C CNN
-	1    6500 3700
-	1    0    0    -1
-$EndComp
 Wire Wire Line
 	6500 3300 6500 3350
@@
 Wire Wire Line
 	6600 3950 6500 3950
-Connection ~ 6500 2550
 $Comp
 L Device:C_Small C6
@@
 Wire Wire Line
 	5900 2200 6750 2200
-$Comp
-L power:+1V8 #PWR05
-U 1 1 5FE12CAB
-P 5650 2200
-F 0 "#PWR05" H 5650 2050 50  0001 C CNN
-F 1 "+1V8" H 5650 2350 50  0000 C CNN
-F 2 "" H 5650 2200 50  0001 C CNN
-F 3 "" H 5650 2200 50  0001 C CNN
-	1    5650 2200
-	1    0    0    -1
-$EndComp
-Connection ~ 5650 2200
 Text GLabel 6750 1850 0    50   Input ~ 0
 VDDPLL
@@
 Wire Wire Line
 	5850 850  5850 800
-$Comp
-L power:+1V8 #PWR07
-U 1 1 5FE1CDDB
-P 5850 800
-F 0 "#PWR07" H 5850 650 50  0001 C CNN
-F 1 "+1V8" H 5850 950 50  0000 C CNN
-F 2 "" H 5850 800 50  0001 C CNN
-F 3 "" H 5850 800 50  0001 C CNN
-	1    5850 800
-	1    0    0    -1
-$EndComp
-$Comp
-L power:+1V8 #PWR01
-U 1 1 5FE1D0E3
-P 5100 800
-F 0 "#PWR01" H 5100 650 50  0001 C CNN
-F 1 "+1V8" H 5100 950 50  0000 C CNN
-F 2 "" H 5100 800 50  0001 C CNN
-F 3 "" H 5100 800 50  0001 C CNN
-	1    5100 800
-	1    0    0    -1
-$EndComp
-$Comp
-L power:+1V8 #PWR03
-U 1 1 5FE1D334
-P 5450 800
-F 0 "#PWR03" H 5450 650 50  0001 C CNN
-F 1 "+1V8" H 5450 950 50  0000 C CNN
-F 2 "" H 5450 800 50  0001 C CNN
-F 3 "" H 5450 800 50  0001 C CNN
-	1    5450 800
-	1    0    0    -1
-$EndComp
 Text GLabel 5450 850  2    50   Input ~ 0
 VDDPLL
@@
 	3250 550  3250 6200
 Text Notes 550  6150 0    50   ~ 0
-BL Generator & SPI FLASH supply voltage
+Main power
 $Comp
 L Regulator_Linear:AZ1117-1.8 U3
@@
 $EndComp
 Text Notes 550  3850 0    50   ~ 0
-Main CPU power reg
+Create 1.8V for the lcd
 $Comp
 L Device:C_Small C?
@@
 Text Notes 13550 2100 0    50   ~ 0
 4GB Flash module using SPI & SD Card protocol
+$Comp
+L Device:LED_Small D?
+U 1 1 5FEB20A3
+P 4800 3200
+F 0 "D?" V 4846 3130 50  0000 R CNN
+F 1 "+3.3v" V 4755 3130 50  0000 R CNN
+F 2 "LED_SMD:LED_0603_1608Metric" V 4800 3200 50  0001 C CNN
+F 3 "~" V 4800 3200 50  0001 C CNN
+	1    4800 3200
+	0    -1   -1   0
+$EndComp
+$Comp
+L power:GND #PWR?
+U 1 1 5FEB20A9
+P 4800 3350
+F 0 "#PWR?" H 4800 3100 50  0001 C CNN
+F 1 "GND" H 4805 3177 50  0000 C CNN
+F 2 "" H 4800 3350 50  0001 C CNN
+F 3 "" H 4800 3350 50  0001 C CNN
+	1    4800 3350
+	1    0    0    -1
+$EndComp
+$Comp
+L Device:R_Small R?
+U 1 1 5FEB20AF
+P 4800 2950
+F 0 "R?" H 4859 2996 50  0000 L CNN
+F 1 "8" H 4859 2905 50  0000 L CNN
+F 2 "Resistor_SMD:R_0603_1608Metric" H 4800 2950 50  0001 C CNN
+F 3 "~" H 4800 2950 50  0001 C CNN
+	1    4800 2950
+	1    0    0    -1
+$EndComp
+Wire Wire Line
+	4800 3050 4800 3100
+Wire Wire Line
+	4800 3300 4800 3350
+Wire Wire Line
+	4800 2850 4800 2800
+$Comp
+L power:+3.3V #PWR?
+U 1 1 5FEB20B8
+P 4800 2800
+F 0 "#PWR?" H 4800 2650 50  0001 C CNN
+F 1 "+3.3V" H 4815 2973 50  0000 C CNN
+F 2 "" H 4800 2800 50  0001 C CNN
+F 3 "" H 4800 2800 50  0001 C CNN
+	1    4800 2800
+	1    0    0    -1
+$EndComp
+$Comp
+L power:+3.3V #PWR?
+U 1 1 5FEBDF98
+P 5650 2200
+F 0 "#PWR?" H 5650 2050 50  0001 C CNN
+F 1 "+3.3V" H 5665 2373 50  0000 C CNN
+F 2 "" H 5650 2200 50  0001 C CNN
+F 3 "" H 5650 2200 50  0001 C CNN
+	1    5650 2200
+	1    0    0    -1
+$EndComp
+Connection ~ 5650 2200
+$Comp
+L power:+3.3V #PWR?
+U 1 1 5FEBE273
+P 6500 2550
+F 0 "#PWR?" H 6500 2400 50  0001 C CNN
+F 1 "+3.3V" H 6350 2650 50  0000 C CNN
+F 2 "" H 6500 2550 50  0001 C CNN
+F 3 "" H 6500 2550 50  0001 C CNN
+	1    6500 2550
+	1    0    0    -1
+$EndComp
+Connection ~ 6500 2550
+$Comp
+L power:+3.3V #PWR?
+U 1 1 5FEBE4C5
+P 6500 2900
+F 0 "#PWR?" H 6500 2750 50  0001 C CNN
+F 1 "+3.3V" H 6350 3000 50  0000 C CNN
+F 2 "" H 6500 2900 50  0001 C CNN
+F 3 "" H 6500 2900 50  0001 C CNN
+	1    6500 2900
+	1    0    0    -1
+$EndComp
+$Comp
+L power:+3.3V #PWR?
+U 1 1 5FEBE61F
+P 6500 3300
+F 0 "#PWR?" H 6500 3150 50  0001 C CNN
+F 1 "+3.3V" H 6350 3350 50  0000 C CNN
+F 2 "" H 6500 3300 50  0001 C CNN
+F 3 "" H 6500 3300 50  0001 C CNN
+	1    6500 3300
+	1    0    0    -1
+$EndComp
+$Comp
+L power:+3.3V #PWR?
+U 1 1 5FEBE7BC
+P 6500 3700
+F 0 "#PWR?" H 6500 3550 50  0001 C CNN
+F 1 "+3.3V" H 6350 3800 50  0000 C CNN
+F 2 "" H 6500 3700 50  0001 C CNN
+F 3 "" H 6500 3700 50  0001 C CNN
+	1    6500 3700
+	1    0    0    -1
+$EndComp
+$Comp
+L power:+3.3V #PWR?
+U 1 1 5FEBF4D3
+P 5100 800
+F 0 "#PWR?" H 5100 650 50  0001 C CNN
+F 1 "+3.3V" H 5115 973 50  0000 C CNN
+F 2 "" H 5100 800 50  0001 C CNN
+F 3 "" H 5100 800 50  0001 C CNN
+	1    5100 800
+	1    0    0    -1
+$EndComp
+$Comp
+L power:+3.3V #PWR?
+U 1 1 5FEBF847
+P 5450 800
+F 0 "#PWR?" H 5450 650 50  0001 C CNN
+F 1 "+3.3V" H 5465 973 50  0000 C CNN
+F 2 "" H 5450 800 50  0001 C CNN
+F 3 "" H 5450 800 50  0001 C CNN
+	1    5450 800
+	1    0    0    -1
+$EndComp
+$Comp
+L power:+3.3V #PWR?
+U 1 1 5FEBFA5B
+P 5850 800
+F 0 "#PWR?" H 5850 650 50  0001 C CNN
+F 1 "+3.3V" H 5865 973 50  0000 C CNN
+F 2 "" H 5850 800 50  0001 C CNN
+F 3 "" H 5850 800 50  0001 C CNN
+	1    5850 800
+	1    0    0    -1
+$EndComp
 $EndSCHEMATC
