File: iPod nano 6 LCD.sch (KiCad schematic (older format))
At the start: 53 parts, among them J1 Molex_503548-1220, J2 USB_C_Receptacle_USB2.0, J3 Conn_01x06_Male, U1 AP5724, U2 ATSAM3SD8BA-AU, U3 AZ1117-1.8, U4 TPS63001, U5 XTSD04GLGEAG, Y1 32.768k, Y2 20MHz

Commit message: Remove the ARM on board.. Going with an fpga...
Parts:
- removed U2: ATSAM3SD8BA-AU, iPod nano 6 LCD:QFP-64_12x12_Pitch0.5mm, symbol iPod~nano~6~LCD:ATSAM3SD8BA-AU
Changed lines of the file:
@@
 Display connector
-$Comp
-L iPod~nano~6~LCD:ATSAM3SD8BA-AU U2
-U 1 1 5FD74BEF
-P 8000 3000
-F 0 "U2" H 8150 -650 50  0000 L CNN
-F 1 "ATSAM3SD8BA-AU" H 7600 -750 50  0000 L CNN
-F 2 "iPod nano 6 LCD:QFP-64_12x12_Pitch0.5mm" H 8000 3000 50  0001 C CNN
-F 3 "" H 8000 3000 50  0001 C CNN
-	1    8000 3000
-	1    0    0    -1
-$EndComp
 $Comp
 L Device:C_Small C7

Commit message: Connecting up the power for the ice40 FPGA I decided to go with.
Parts:
- removed L3: 2.2uH, Inductor_SMD:L_0603_1608Metric, symbol Device:L
- removed U3: AZ1117-1.8, Package_TO_SOT_SMD:SOT-223-3_TabPin2, symbol Regulator_Linear:AZ1117-1.8
- removed U4: TPS63001, Package_SON:Texas_DRC0010J_ThermalVias, symbol Regulator_Switching:TPS63002
- added C22, C23, C24, C25, C26, C30, C31, C32, C33, C? (x4): 1u, Capacitor_SMD:C_0603_1608Metric, symbol Device:C_Small
- added C27: DNP, Capacitor_SMD:C_0603_1608Metric, symbol Device:C_Small
- added C28: 10u, Capacitor_SMD:C_0603_1608Metric, symbol Device:C_Small
- added C29: 100n, Capacitor_SMD:C_0603_1608Metric, symbol Device:C_Small
- added D6: ~~800mVf, Diode_SMD:D_0603_1608Metric, symbol Device:D_Small
- added L2, L3, L4: 2.2u, Inductor_SMD:L_0603_1608Metric, symbol Device:L_Small
- added R16, R18, R19, R20: 100k, Resistor_SMD:R_0603_1608Metric, symbol Device:R_Small
- added R17: 200k, Resistor_SMD:R_0603_1608Metric, symbol Device:R_Small
- added R21: 100, Resistor_SMD:R_0603_1608Metric, symbol Device:R_Small
- added R22: 2k2, Resistor_SMD:R_0603_1608Metric, symbol Device:R_Small
- added R23: 10k, Resistor_SMD:R_0603_1608Metric, symbol Device:R_Small
- added TP1: 1.8v, TestPoint:TestPoint_Pad_D1.0mm, symbol Connector:TestPoint
- added TP2: 3.3v, TestPoint:TestPoint_Pad_D1.0mm, symbol Connector:TestPoint
- added TP3: 1.2v, TestPoint:TestPoint_Pad_D1.0mm, symbol Connector:TestPoint
- added U2: ICE40HX1K-TQ144, Package_QFP:TQFP-144_20x20mm_P0.5mm, symbol iPod~nano~6~LCD:ICE40HX1K-TQ144
- added U3, U4, U6: TLV62569DBV, Package_TO_SOT_SMD:SOT-23-5, symbol Regulator_Switching:TLV62569DBV
- C10, C12, C14, C5, C6, C7, C9: value 1u -> 10u
- C11, C3, C8: value 1u -> 4.7u
- C15: value .1u -> 10u
- C17: value 10u -> 1u
- R3: value 100 -> 442k
- gave numbers to parts that had none: 2
Connections:
- net labels added: +1V2, +3V3, GNDPLL, VCCPLL, VCC_SPI, VPP_2V5
- wire segments 175 -> 285
Other:
- note removed: "Create 1.8V for the lcd"
- note removed: "Main power"
- moved on the sheet: J2, J3

Commit message: Add config SPI and silkscreen for lcd
Parts:
- removed C13, C18: 12.5p, Capacitor_SMD:C_0603_1608Metric, symbol Device:C_Small
- removed C19, C20: 10p, Capacitor_SMD:C_0603_1608Metric, symbol Device:C_Small
- removed Y1: 32.768k, Crystal:Crystal_SMD_Abracon_ABS25-4Pin_8.0x3.8mm, symbol Device:Crystal_Small
- removed Y2: 20MHz, Crystal:Crystal_SMD_Abracon_ABM8G-4Pin_3.2x2.5mm, symbol Device:Crystal_Small
- added C38: 1u, Capacitor_SMD:C_0603_1608Metric, symbol Device:C_Small
- added U7: AT25xxx, Package_DFN_QFN:DFN-8-1EP_3x2mm_P0.5mm_EP1.75x1.45mm, symbol Memory_EEPROM:AT25xxx
- gave numbers to parts that had none: 4
Connections:
- net labels added: CFG_CS, SCK
- wire segments 285 -> 268
Changed lines of the file:
@@
 Text GLabel 6250 8700 2    50   Input ~ 0
 TDI
-Text GLabel 8400 5700 2    50   Input ~ 0
-TMS
-Text GLabel 8400 5500 2    50   Input ~ 0
-TDI
-Text GLabel 8400 5600 2    50   Input ~ 0
-TDO
-Text GLabel 8400 5800 2    50   Input ~ 0
-TCK
 $Comp
 L power:GND #PWR?
@@
 	1    0    0    -1
 $EndComp
-$Comp
-L Device:Crystal_Small Y1
-U 1 1 5FF05C66
-P 8750 2450
-F 0 "Y1" V 8704 2538 50  0000 L CNN
-F 1 "32.768k" V 8900 2300 50  0000 L CNN
-F 2 "Crystal:Crystal_SMD_Abracon_ABS25-4Pin_8.0x3.8mm" H 8750 2450 50  0001 C CNN
-F 3 "~" H 8750 2450 50  0001 C CNN
-	1    8750 2450
-	0    1    1    0
-$EndComp
-Wire Wire Line
-	8500 2400 8500 2350
-Wire Wire Line
-	8500 2350 8750 2350
-Wire Wire Line
-	8400 2400 8500 2400
-Wire Wire Line
-	8400 2500 8500 2500
-Wire Wire Line
-	8500 2500 8500 2550
-Wire Wire Line
-	8500 2550 8750 2550
-Connection ~ 8750 2350
-Connection ~ 8750 2550
-$Comp
-L Device:C_Small C13
-U 1 1 5FF208F8
-P 9050 2350
-F 0 "C13" H 8959 2304 50  0000 R CNN
-F 1 "12.5p" H 8959 2395 50  0000 R CNN
-F 2 "Capacitor_SMD:C_0603_1608Metric" H 9050 2350 50  0001 C CNN
-F 3 "~" H 9050 2350 50  0001 C CNN
-	1    9050 2350
-	0    -1   1    0
-$EndComp
-$Comp
-L Device:C_Small C18
-U 1 1 5FF20D1C
-P 9050 2550
-F 0 "C18" H 8959 2504 50  0000 R CNN
-F 1 "12.5p" H 8959 2595 50  0000 R CNN
-F 2 "Capacitor_SMD:C_0603_1608Metric" H 9050 2550 50  0001 C CNN
-F 3 "~" H 9050 2550 50  0001 C CNN
-	1    9050 2550
-	0    -1   -1   0
-$EndComp
-Wire Wire Line
-	8750 2350 8950 2350
-Wire Wire Line
-	8950 2550 8750 2550
-Wire Wire Line
-	9150 2550 9200 2550
-Wire Wire Line
-	9200 2550 9200 2350
-Wire Wire Line
-	9200 2350 9150 2350
-$Comp
-L power:GND #PWR0116
-U 1 1 5FF353AF
-P 9200 2550
-F 0 "#PWR0116" H 9200 2300 50  0001 C CNN
-F 1 "GND" H 9300 2450 50  0000 C CNN
-F 2 "" H 9200 2550 50  0001 C CNN
-F 3 "" H 9200 2550 50  0001 C CNN
-	1    9200 2550
-	1    0    0    -1
-$EndComp
-Connection ~ 9200 2550
-$Comp
-L Device:Crystal_Small Y2
-U 1 1 5FF4687B
-P 8750 5950
-F 0 "Y2" V 8704 6038 50  0000 L CNN
-F 1 "20MHz" V 8900 5800 50  0000 L CNN
-F 2 "Crystal:Crystal_SMD_Abracon_ABM8G-4Pin_3.2x2.5mm" H 8750 5950 50  0001 C CNN
-F 3 "~" H 8750 5950 50  0001 C CNN
-	1    8750 5950
-	0    1    1    0
-$EndComp
-Wire Wire Line
-	8500 5900 8500 5850
-Wire Wire Line
-	8500 5850 8750 5850
-Wire Wire Line
-	8400 5900 8500 5900
-Wire Wire Line
-	8400 6000 8500 6000
-Wire Wire Line
-	8500 6000 8500 6050
-Wire Wire Line
-	8500 6050 8750 6050
-Connection ~ 8750 5850
-Connection ~ 8750 6050
-$Comp
-L Device:C_Small C19
-U 1 1 5FF46889
-P 9050 5850
-F 0 "C19" H 8959 5804 50  0000 R CNN
-F 1 "10p" H 8959 5895 50  0000 R CNN
-F 2 "Capacitor_SMD:C_0603_1608Metric" H 9050 5850 50  0001 C CNN
-F 3 "~" H 9050 5850 50  0001 C CNN
-	1    9050 5850
-	0    -1   1    0
-$EndComp
-$Comp
-L Device:C_Small C20
-U 1 1 5FF4688F
-P 9050 6050
-F 0 "C20" H 8959 6004 50  0000 R CNN
-F 1 "10p" H 8959 6095 50  0000 R CNN
-F 2 "Capacitor_SMD:C_0603_1608Metric" H 9050 6050 50  0001 C CNN
-F 3 "~" H 9050 6050 50  0001 C CNN
-	1    9050 6050
-	0    -1   -1   0
-$EndComp
-Wire Wire Line
-	8750 5850 8950 5850
-Wire Wire Line
-	8950 6050 8750 6050
-Wire Wire Line
-	9150 6050 9200 6050
-Wire Wire Line
-	9200 6050 9200 5850
-Wire Wire Line
-	9200 5850 9150 5850
-$Comp
-L power:GND #PWR020
-U 1 1 5FF4689A
-P 9200 6050
-F 0 "#PWR020" H 9200 5800 50  0001 C CNN
-F 1 "GND" H 9300 5950 50  0000 C CNN
-F 2 "" H 9200 6050 50  0001 C CNN
-F 3 "" H 9200 6050 50  0001 C CNN
-	1    9200 6050
-	1    0    0    -1
-$EndComp
-Connection ~ 9200 6050
 $Comp
 L iPod~nano~6~LCD:XTSD04GLGEAG U5
@@
 $EndComp
 $Comp
-L Device:C_Small C?
+L Device:C_Small C37
 U 1 1 60640315
 P 12450 6100
-F 0 "C?" H 12359 6054 50  0000 R CNN
+F 0 "C37" H 12359 6054 50  0000 R CNN
 F 1 "1u" H 12359 6145 50  0000 R CNN
 F 2 "Capacitor_SMD:C_0603_1608Metric" H 12450 6100 50  0001 C CNN
@@
 	12200 6100 12200 5950
 $Comp
-L Device:C_Small C?
+L Device:C_Small C36
 U 1 1 606A68A3
 P 11300 4250
-F 0 "C?" H 11209 4204 50  0000 R CNN
+F 0 "C36" H 11209 4204 50  0000 R CNN
 F 1 "1u" H 11209 4295 50  0000 R CNN
 F 2 "Capacitor_SMD:C_0603_1608Metric" H 11300 4250 50  0001 C CNN
@@
 	11050 4250 11050 4100
 $Comp
-L Device:C_Small C?
+L Device:C_Small C34
 U 1 1 6071123E
 P 10050 6750
-F 0 "C?" H 9959 6704 50  0000 R CNN
+F 0 "C34" H 9959 6704 50  0000 R CNN
 F 1 "1u" H 9959 6795 50  0000 R CNN
 F 2 "Capacitor_SMD:C_0603_1608Metric" H 10050 6750 50  0001 C CNN
@@
 	11450 900  11450 1050
 $Comp
-L Device:C_Small C?
+L Device:C_Small C35
 U 1 1 607837B2
 P 11250 1050
-F 0 "C?" H 11159 1004 50  0000 R CNN
+F 0 "C35" H 11159 1004 50  0000 R CNN
 F 1 "1u" H 11159 1095 50  0000 R CNN
 F 2 "Capacitor_SMD:C_0603_1608Metric" H 11250 1050 50  0001 C CNN
@@
 Wire Wire Line
 	11000 1050 11000 900
+$Comp
+L power:GND #PWR042
+U 1 1 607F02CC
+P 1375 8625
+F 0 "#PWR042" H 1375 8375 50  0001 C CNN
+F 1 "GND" H 1380 8452 50  0000 C CNN
+F 2 "" H 1375 8625 50  0001 C CNN
+F 3 "" H 1375 8625 50  0001 C CNN
+	1    1375 8625
+	1    0    0    -1
+$EndComp
+$Comp
+L power:GND #PWR?
+U 1 1 6081C3F1
+P 1825 7975
+AR Path="/5FEB2752/6081C3F1" Ref="#PWR?"  Part="1"
+AR Path="/6081C3F1" Ref="#PWR043"  Part="1"
+F 0 "#PWR043" H 1825 7725 50  0001 C CNN
+F 1 "GND" H 1830 7802 50  0000 C CNN
+F 2 "" H 1825 7975 50  0001 C CNN
+F 3 "" H 1825 7975 50  0001 C CNN
+	1    1825 7975
+	1    0    0    -1
+$EndComp
+$Comp
+L Device:C_Small C38
+U 1 1 607F1BE9
+P 1575 7950
+F 0 "C38" H 1484 7904 50  0000 R CNN
+F 1 "1u" H 1484 7995 50  0000 R CNN
+F 2 "Capacitor_SMD:C_0603_1608Metric" H 1575 7950 50  0001 C CNN
+F 3 "~" H 1575 7950 50  0001 C CNN
+	1    1575 7950
+	0    1    1    0
+$EndComp
+$Comp
+L Memory_EEPROM:AT25xxx U7
+U 1 1 607EEFB8
+P 1375 8325
+F 0 "U7" H 1075 8850 50  0000 C CNN
+F 1 "AT25xxx" H 1175 8750 50  0000 C CNN
+F 2 "Package_DFN_QFN:DFN-8-1EP_3x2mm_P0.5mm_EP1.75x1.45mm" H 1375 8325 50  0001 C CNN
+F 3 "http://ww1.microchip.com/downloads/en/DeviceDoc/Atmel-8707-SEEPROM-AT25010B-020B-040B-Datasheet.pdf" H 1375 8325 50  0001 C CNN
+	1    1375 8325
+	1    0    0    -1
+$EndComp
+Wire Wire Line
+	1675 7950 1825 7950
+Wire Wire Line
+	1825 7950 1825 7975
+Wire Wire Line
+	1375 7950 1475 7950
+Wire Wire Line
+	1375 7950 1375 8025
+$Comp
+L power:+3.3V #PWR041
+U 1 1 60875906
+P 1375 7875
+F 0 "#PWR041" H 1375 7725 50  0001 C CNN
+F 1 "+3.3V" H 1390 8048 50  0000 C CNN
+F 2 "" H 1375 7875 50  0001 C CNN
+F 3 "" H 1375 7875 50  0001 C CNN
+	1    1375 7875
+	1    0    0    -1
+$EndComp
+Connection ~ 1375 7950
+Wire Wire Line
+	1375 7875 1375 7950
+Text GLabel 14100 3800 0    50   Input ~ 0
+SCK
+Text GLabel 14100 3900 0    50   Input ~ 0
+CFG_CS
+Text GLabel 1775 8225 2    50   Input ~ 0
+SCK
+Text GLabel 975  8425 0    50   Input ~ 0
+CFG_CS
+Text GLabel 14100 3600 0    50   Input ~ 0
+MOSI
+Text GLabel 14100 3700 0    50   Input ~ 0
+MISO
+Text GLabel 1775 8325 2    50   Input ~ 0
+MOSI
+Text GLabel 1775 8425 2    50   Input ~ 0
+MISO
 $EndSCHEMATC

Commit message: Add LCD differential pairs, user led and reset/user butons, connect SD module CS pin to FPGA
Parts:
- removed C1, C2, C4: 1u, Capacitor_SMD:C_0603_1608Metric, symbol Device:C_Small
- removed J3: Conn_01x06_Male, Connector_JST:JST_GH_BM06B-GHS-TBT_1x06-1MP_P1.25mm_Vertical, symbol Connector_Generic_MountingPin:Conn_01x06_MountingPin
- added C13, C39, C40, C43, C44, C46: 100n, Capacitor_SMD:C_0603_1608Metric, symbol Device:C_Small
- added C18, C41, C42, C45: 4.7u, Capacitor_SMD:C_0603_1608Metric, symbol Device:C_Small
- added C19, C20: 10p, Capacitor_SMD:C_0603_1608Metric, symbol Device:C_Small
- added D7, D8: USR, LED_SMD:LED_0603_1608Metric, symbol Device:LED_Small
- added L5, L6: 600, Inductor_SMD:L_0603_1608Metric, symbol Device:L_Small
- added R24: 1M, Resistor_SMD:R_0603_1608Metric, symbol Device:R_Small
- added R25, R26: 5.1k, Resistor_SMD:R_0603_1608Metric, symbol Device:R_Small
- added R27, R28: 12k, Resistor_SMD:R_0603_1608Metric, symbol Device:R_Small
- added R29, R31, R32, R34: 10k, Resistor_SMD:R_0603_1608Metric, symbol Device:R_Small
- added R30: 2k2, Resistor_SMD:R_0603_1608Metric, symbol Device:R_Small
- added R33: 220, Resistor_SMD:R_0603_1608Metric, symbol Device:R_Small
- added SW1, SW2: SW_Push, Button_Switch_SMD:SW_Push_1P1T_NO_CK_KMR2, symbol Switch:SW_Push
- added U8: USBLC6-2P6, Package_TO_SOT_SMD:SOT-666, symbol Power_Protection:USBLC6-2P6
- added U9: FT232H, Package_DFN_QFN:QFN-48-1EP_8x8mm_P0.5mm_EP6.2x6.2mm_ThermalVias, symbol Interface_USB:FT232H
- added Y1: 12MHz, Crystal:Crystal_SMD_Abracon_ABM8G-4Pin_3.2x2.5mm, symbol Device:Crystal_Small
- R8: value 220 -> 8
Connections:
- net labels added: ICE_CN, ICE_CNBIAS, ICE_CP, ICE_CPBIAS, ICE_CRESET, ICE_DN, ICE_DNBIAS, ICE_DONE, ICE_DP, ICE_DPBIAS, ICE_SS_B, LCD_CN, LCD_CP, LCD_DN, LCD_DP, USBD_N, USBD_P, USR_LED, VSYNC
- net labels removed: CLKN, CLKP, DN, DP, IC_CLKN, IC_CLKP, SCLK, SYNC, TCK, TDI, TDO, TMS, VDDIN, VDDOUT, VDDPLL
- wire segments 268 -> 401
Other:
- note added: "1%"
- note removed: "Some of the CPU decoupling\n"
- moved on the sheet: C10, C11, C12, C14, C15, C16, C3, C33, C37, C38, C5, C6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

Commit message: SPI line pullups
Parts:
- added R35, R36, R37, R?: 10k, Resistor_SMD:R_0603_1608Metric, symbol Device:R_Small
Connections:
- wire segments 401 -> 414
Changed lines of the file:
@@
+	1    0    0    -1
+$EndComp
+$Comp
+L Device:R_Small R35
+U 1 1 5FF851C5
+P 8175 9225
+F 0 "R35" V 8250 9200 50  0000 L CNN
+F 1 "10k" V 8250 9025 50  0000 L CNN
+F 2 "Resistor_SMD:R_0603_1608Metric" H 8175 9225 50  0001 C CNN
+F 3 "~" H 8175 9225 50  0001 C CNN
+	1    8175 9225
+	1    0    0    -1
+$EndComp
+$Comp
+L Device:R_Small R36
+U 1 1 5FF85391
+P 8350 9225
+F 0 "R36" V 8425 9200 50  0000 L CNN
+F 1 "10k" V 8425 9025 50  0000 L CNN
+F 2 "Resistor_SMD:R_0603_1608Metric" H 8350 9225 50  0001 C CNN
+F 3 "~" H 8350 9225 50  0001 C CNN
+	1    8350 9225
+	1    0    0    -1
+$EndComp
+$Comp
+L Device:R_Small R37
+U 1 1 5FF8559D
+P 8525 9225
+F 0 "R37" V 8600 9200 50  0000 L CNN
+F 1 "10k" V 8600 9025 50  0000 L CNN
+F 2 "Resistor_SMD:R_0603_1608Metric" H 8525 9225 50  0001 C CNN
+F 3 "~" H 8525 9225 50  0001 C CNN
+	1    8525 9225
+	1    0    0    -1
+$EndComp
+Wire Wire Line
+	7750 9425 8175 9425
+Wire Wire Line
+	8175 9425 8175 9325
+Wire Wire Line
+	7750 9525 8350 9525
+Wire Wire Line
+	8350 9525 8350 9325
+Wire Wire Line
+	7750 9625 8525 9625
+Wire Wire Line
+	8525 9625 8525 9325
+Wire Wire Line
+	8175 9125 8175 9075
+Wire Wire Line
+	8175 9075 8350 9075
+Wire Wire Line
+	8525 9075 8525 9125
+Wire Wire Line
+	8350 9125 8350 9075
+Connection ~ 8350 9075
+Wire Wire Line
+	8350 9075 8525 9075
+$Comp
+L power:+3.3V #PWR0130
+U 1 1 6006DFC2
+P 8350 9075
+F 0 "#PWR0130" H 8350 8925 50  0001 C CNN
+F 1 "+3.3V" H 8365 9248 50  0000 C CNN
+F 2 "" H 8350 9075 50  0001 C CNN
+F 3 "" H 8350 9075 50  0001 C CNN
+	1    8350 9075
+	1    0    0    -1
+$EndComp
+$Comp
+L Device:R_Small R?
+U 1 1 60086DC7
+P 13875 1175
+F 0 "R?" V 13950 1150 50  0000 L CNN
+F 1 "10k" V 13950 975 50  0000 L CNN
+F 2 "Resistor_SMD:R_0603_1608Metric" H 13875 1175 50  0001 C CNN
+F 3 "~" H 13875 1175 50  0001 C CNN
+	1    13875 1175
+	1    0    0    -1
+$EndComp
+Wire Wire Line
+	14550 1300 13875 1300
+Wire Wire Line
+	13875 1300 13875 1275
+$Comp
+L power:+3.3V #PWR?
+U 1 1 600B6B09
+P 13875 1075
+F 0 "#PWR?" H 13875 925 50  0001 C CNN
+F 1 "+3.3V" H 13890 1248 50  0000 C CNN
+F 2 "" H 13875 1075 50  0001 C CNN
+F 3 "" H 13875 1075 50  0001 C CNN
+	1    13875 1075
 	1    0    0    -1
 $EndComp

Commit message: Debounce cap for user switch
Parts:
- added C?: 10u, Capacitor_SMD:C_0603_1608Metric, symbol Device:C_Small
- gave numbers to parts that had none: 1
Connections:
- wire segments 414 -> 415
Changed lines of the file:
@@
 $EndComp
 $Comp
-L Device:R_Small R?
+L Device:R_Small R38
 U 1 1 60086DC7
 P 13875 1175
-F 0 "R?" V 13950 1150 50  0000 L CNN
+F 0 "R38" V 13950 1150 50  0000 L CNN
 F 1 "10k" V 13950 975 50  0000 L CNN
 F 2 "Resistor_SMD:R_0603_1608Metric" H 13875 1175 50  0001 C CNN
@@
 	13875 1300 13875 1275
 $Comp
-L power:+3.3V #PWR?
+L power:+3.3V #PWR0131
 U 1 1 600B6B09
 P 13875 1075
-F 0 "#PWR?" H 13875 925 50  0001 C CNN
+F 0 "#PWR0131" H 13875 925 50  0001 C CNN
 F 1 "+3.3V" H 13890 1248 50  0000 C CNN
 F 2 "" H 13875 1075 50  0001 C CNN
@@
 	1    0    0    -1
 $EndComp
+$Comp
+L Device:C_Small C?
+U 1 1 600D356B
+P 8925 8150
+AR Path="/5FEB2752/600D356B" Ref="C?"  Part="1"
+AR Path="/600D356B" Ref="C?"  Part="1"
+F 0 "C?" H 9017 8196 50  0000 L CNN
+F 1 "10u" H 9017 8105 50  0000 L CNN
+F 2 "Capacitor_SMD:C_0603_1608Metric" H 8925 8150 50  0001 C CNN
+F 3 "~" H 8925 8150 50  0001 C CNN
+	1    8925 8150
+	-1   0    0    -1
+$EndComp
+Wire Wire Line
+	8925 8000 8925 8050
+$Comp
+L power:GND #PWR?
+U 1 1 601044B4
+P 8925 8250
+F 0 "#PWR?" H 8925 8000 50  0001 C CNN
+F 1 "GND" H 8930 8077 50  0000 C CNN
+F 2 "" H 8925 8250 50  0001 C CNN
+F 3 "" H 8925 8250 50  0001 C CNN
+	1    8925 8250
+	1    0    0    -1
+$EndComp

Commit message: Start schematic cleanup
Parts:
- gave numbers to parts that had none: 1
Connections:
- net labels added: LCD_RESET
- wire segments 415 -> 433
Other:
- note added: "2V5, PLL and SPI power\n"
- note added: "4GB Flash module using SPI with SD Card protocol"
- note added: "Display signal and bias resistors\n"
- note added: "FPGA Housekeeping and config pins"
- note added: "IOB\nUSER pushbutton and SD Flash CS Pin\n"
- note added: "IOR\nUSER LED"
- note added: "IOT\nLCD communications"
- note added: "Main power bus dc-dc's\n"
- note added: "POWER, USER, DONE LEDs (DONE has resistor elsewhere)"
- note added: "USB -> SPI flash programmer, schematic from Greg Davill's JTAG programmer, adapted with ICEBreaker board schematic\n"
- note added: "Unused but powered IOL.\nLeft in to be used for scope probing if needed"
- note added: "ice40 config flash"
- note removed: "4GB Flash module using SPI & SD Card protocol"
- moved on the sheet: C1, C10, C11, C12, C14, C15, C17, C21, C22, C23, C24, C25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

Commit message: Adjust pin mapping a bit.
Connections:
- wire segments 433 -> 432
Changed lines of the file:
@@
 Text Label 14375 4300 0    50   ~ 0
 ICE_DPBIAS
+Text Label 12625 3125 2    50   ~ 0
+ICE_DP
 Text Label 12625 3025 2    50   ~ 0
-ICE_DP
-Text Label 12625 3125 2    50   ~ 0
 ICE_DPBIAS
 Text Label 12625 3225 2    50   ~ 0
@@
 Text Label 15275 4675 2    50   ~ 0
 LCD_CN
+Text Label 12625 3525 2    50   ~ 0
+ICE_CN
 Text Label 12625 3425 2    50   ~ 0
-ICE_CN
-Text Label 12625 3525 2    50   ~ 0
 ICE_CNBIAS
 Text Label 12625 3625 2    50   ~ 0
@@
 Wire Wire Line
 	15150 3025 15100 3025
-Wire Wire Line
-	12625 3925 12575 3925
-Text Label 12575 3925 2    50   ~ 0
+Text Label 12625 3925 2    50   ~ 0
 LCD_RESET
 Wire Wire Line
